Commit message: Automate 2022 Integration (#5)
* Remove temporary erase of first and last raster

* Converted application window to widget

* Update planning functions to not be blocking

* Add Rviz panel for SNP application

* Renamed rosconwindow to snp_widget

* Changed launch files to use rviz panel version of application

* Added ROI selection mesh modifier and widget

* Added noether plugin for ROI mesh modifier

* Add TPP widget

* Added TPP app

* Updated launch file to start TPP app instead of node

* Updated Rviz config

* Remove TPP parameter from service definition; added string for mesh frame to TPP service defintion; updated existing TPP nodes

* Transform selection into mesh frame

* Changed namespace from snp to snp_tpp

* Created unique names for transition commands

* Async callback for motion execution

* fixup tpp widget header

* Faster scan traj

* Automate setup camera calibration

* Updated LVS to ensure at least 5 wps

* Updated the rviz config file

* Added collision geometry for TCP

* Updated dependencies and README

* Updated TPP to use latest version of noether_gui

* Ran CMake format

* Ran clang format

* Replaced references to open3d_interface

* Updated .repos files

* Added xmlrpcpp dependency for CI

File: snp_support/urdf/workcell.xacro (robot description, xacro)
@@ -117,4 +117,10 @@
       </geometry>
     </collision>
+    <collision name="tcp">
+      <geometry>
+        <cylinder radius="${1.5 * 0.0254}" length="${2.0 * 0.0254}"/>
+      </geometry>
+      <origin xyz="${-0.263 + 1.5 * 0.0254} 0.0 0.083" rpy="0 ${radians(-90)} 0"/>
+    </collision>
   </link>
   <joint name="tool0_to_ee" type="fixed">
