Commit message: Reorganize application-specific files (#13)
* Combined support and bringup package into single application implementation package

* Removed application-specific instructions from README; replace with general description

* Reverted to update from https://github.com/ros-industrial-consortium/scan_n_plan_workshop/pull/9

* Set planner verbose by default

* Changed name of dependencies file

* Updated documentation

* Updated documentation per review

File: snp_automate_2022/urdf/workcell.xacro (robot description, xacro)
@@ -38,5 +38,5 @@
     <visual>
       <geometry>
-        <mesh filename="package://snp_support/meshes/visual/steel_table.ply"/>
+        <mesh filename="package://snp_automate_2022/meshes/visual/steel_table.ply"/>
       </geometry>
       <material name="dark_gray"/>
@@ -44,5 +44,5 @@
     <collision>
       <geometry>
-        <mesh filename="package://snp_support/meshes/collision/steel_table.ply"/>
+        <mesh filename="package://snp_automate_2022/meshes/collision/steel_table.ply"/>
       </geometry>
     </collision>
@@ -74,45 +74,45 @@
     <visual>
       <geometry>
-        <mesh filename="package://snp_support/meshes/visual/end_effector.stl"/>
+        <mesh filename="package://snp_automate_2022/meshes/visual/end_effector.stl"/>
       </geometry>
     </visual>
     <collision name="compliance">
       <geometry>
-        <mesh filename="package://snp_support/meshes/collision/afd310.ply"/>
+        <mesh filename="package://snp_automate_2022/meshes/collision/afd310.ply"/>
       </geometry>
     </collision>
     <collision name="spindle">
       <geometry>
-        <mesh filename="package://snp_support/meshes/collision/rps100.ply"/>
+        <mesh filename="package://snp_automate_2022/meshes/collision/rps100.ply"/>
       </geometry>
     </collision>
     <collision name="backplate">
       <geometry>
-        <mesh filename="package://snp_support/meshes/collision/backplate.ply"/>
+        <mesh filename="package://snp_automate_2022/meshes/collision/backplate.ply"/>
       </geometry>
     </collision>
     <collision name="frontplate">
       <geometry>
-        <mesh filename="package://snp_support/meshes/collision/front.ply"/>
+        <mesh filename="package://snp_automate_2022/meshes/collision/front.ply"/>
       </geometry>
     </collision>
     <collision name="camera1">
       <geometry>
-        <mesh filename="package://snp_support/meshes/collision/camera1.ply"/>
+        <mesh filename="package://snp_automate_2022/meshes/collision/camera1.ply"/>
       </geometry>
     </collision>
     <collision name="camera2">
       <geometry>
-        <mesh filename="package://snp_support/meshes/collision/camera2.ply"/>
+        <mesh filename="package://snp_automate_2022/meshes/collision/camera2.ply"/>
       </geometry>
     </collision>
     <collision name="sidebracket1">
       <geometry>
-        <mesh filename="package://snp_support/meshes/collision/bracket1.ply"/>
+        <mesh filename="package://snp_automate_2022/meshes/collision/bracket1.ply"/>
       </geometry>
     </collision>
     <collision name="sidebracket2">
       <geometry>
-        <mesh filename="package://snp_support/meshes/collision/bracket2.ply"/>
+        <mesh filename="package://snp_automate_2022/meshes/collision/bracket2.ply"/>
       </geometry>
     </collision>
@@ -128,5 +128,5 @@
     <child link="ee"/>
   </joint>
-  <xacro:property name="camera_cal" value="${load_yaml('$(find snp_support)/config/camera_calibration.yaml')}" />
+  <xacro:property name="camera_cal" value="${load_yaml('$(find snp_automate_2022)/config/camera_calibration.yaml')}" />
   <link name="camera_color_optical_frame"/>
   <joint name="tool0_to_camera" type="fixed">
