Commit message: Humble build (#52)
* Fix templates on declaring parameters

* Fix runtime errors

* Update noether for humble build

* add vtk to rosdep skip

* Updated dependencies to be by ROS version

* Change skip key to just 'libvtk'

* Check ROS version for how params are declared

* Added ROS version check for tf2_eigen include

* Added tf2_eigen depends to various packages

* Added tf2_eigen to planning package CMakeLists

* Fixed a templated declare param previously missed

* Clang formatting

* Clang formatting (pt 2)

* Cleaner ROS version checking

* Set C++ version to 17 for `__has_include` macro

* Removed #if's from different ROS versions

* Fix where things built, but didn't work in humble

* Fix load_yaml difference between foxy and humble+

* Clang formatting

* Update snp_blending support to work with humble

File: snp_blending/urdf/workcell.xacro (robot description, xacro)
@@ -94,5 +94,11 @@
   </joint>
   <!-- Camera Calibration-->
-  <xacro:property name="camera_cal" value="${load_yaml('$(find snp_blending)/config/calibration.yaml')}" />
+  <xacro:arg name="ros_distro" default="humble"/>
+  <xacro:if value="${'$(arg ros_distro)' > 'foxy'}">
+    <xacro:property name="camera_cal" value="${xacro.load_yaml('$(find snp_blending)/config/calibration.yaml')}" />
+  </xacro:if>
+  <xacro:unless value="${'$(arg ros_distro)' > 'foxy'}">
+    <xacro:property name="camera_cal" value="${load_yaml('$(find snp_blending)/config/calibration.yaml')}" />
+  </xacro:unless>
   <link name="camera_color_optical_frame"/>
   <joint name="tool0_to_camera" type="fixed">
@@ -113,5 +119,10 @@
   <xacro:property name="table_width" value="${60*0.0254}"/>
   <xacro:property name="table_length" value="${36*0.0254}"/>
-  <xacro:property name="table_cal" value="${load_yaml('$(find snp_blending)/config/table_calibration.yaml')}" />
+  <xacro:if value="${'$(arg ros_distro)' > 'foxy'}">
+    <xacro:property name="table_cal" value="${xacro.load_yaml('$(find snp_blending)/config/table_calibration.yaml')}" />
+  </xacro:if>
+  <xacro:unless value="${'$(arg ros_distro)' > 'foxy'}">
+    <xacro:property name="table_cal" value="${load_yaml('$(find snp_blending)/config/table_calibration.yaml')}" />
+  </xacro:unless>
   <xacro:cuboid name="table" l="${table_length}" w="${table_width}" h="${table_height}" material="light_gray" offset="True"/>
   <joint name="floor_to_table" type="fixed">
