Commit message: Integration Changes - 5.10.2023 (#24)
* Added updated scan trajectory around the work table

* Added TPP yaml file

* Parameterized TSDF values

* Updated TSDF parameters in launch files for blending and automate demo

* Added calibration files

* Fixed table calibration

* Updated camera calibration

* Updated pointcloud parameter names to the latest realsense nomenclature

* Updated scan trajectory

* Updated tpp configuration

* Updated Pushcorp URDF and TCP location

* Show output from motion planner node on screen

---------

Co-authored-by: Chris Lewis <drchrislewis@gmail.com>

File: snp_blending/urdf/pushcorp.xacro (robot description, xacro)
@@ -3,4 +3,7 @@
   <xacro:macro name="pushcorp" params="prefix">
     <xacro:property name="static_thickness" value="0.0785"/>
+    <xacro:property name="media_radius" value="${2 * 0.0254}"/>
+    <xacro:property name="chuck_length" value="0.055"/>
+    <xacro:property name="chuck_radius" value="${1.0 * 0.0254}}"/>
     <link name="${prefix}base">
       <visual>
@@ -38,13 +41,26 @@
       <!-- Grinding media -->
       <visual>
-        <origin xyz="0.200 0 ${0.190 - static_thickness}" rpy="0 ${radians(90)} 0"/>
+        <origin xyz="${0.200 + chuck_length / 2} 0 ${0.190 - static_thickness}" rpy="0 ${radians(90)} 0"/>
         <geometry>
-          <cylinder radius="0.1" length="0.005"/>
+          <cylinder radius="${chuck_radius}" length="${chuck_length}"/>
         </geometry>
       </visual>
       <collision>
-        <origin xyz="0.200 0 ${0.190 - static_thickness}" rpy="0 ${radians(90)} 0"/>
+        <origin xyz="${0.200 + chuck_length / 2} 0 ${0.190 - static_thickness}" rpy="0 ${radians(90)} 0"/>
         <geometry>
-          <cylinder radius="0.1" length="0.005"/>
+          <cylinder radius="${chuck_radius}" length="${chuck_length}"/>
+        </geometry>
+      </collision>
+      <!-- Grinding media -->
+      <visual>
+        <origin xyz="${0.200 + chuck_length} 0 ${0.190 - static_thickness}" rpy="0 ${radians(90)} 0"/>
+        <geometry>
+          <cylinder radius="${media_radius}" length="0.005"/>
+        </geometry>
+      </visual>
+      <collision>
+        <origin xyz="${0.200 + chuck_length} 0 ${0.190 - static_thickness}" rpy="0 ${radians(90)} 0"/>
+        <geometry>
+          <cylinder radius="${media_radius}" length="0.005"/>
         </geometry>
       </collision>

File: snp_blending/urdf/workcell.xacro (robot description, xacro)
@@ -49,9 +49,9 @@
   <xacro:property name="pushcorp_box_height" value="${30 * 0.0254}"/>
   <xacro:cuboid name="pushcorp_box" l="${pushcorp_box_length}" w="${pushcorp_box_width}" h="${pushcorp_box_height}" material="light_gray"/>
-  <link name="buffy_tcp" />
+  <link name="buffy_tcp"/>
   <joint name="buffy_tcp_joint" type="fixed">
     <parent link="tool0"/>
     <child link="buffy_tcp"/>
-    <origin xyz="0.210 0 0.19" rpy="0 ${pi/2} 0"/>
+    <origin xyz="0.265 0 0.19" rpy="0 ${pi/2} 0"/>
   </joint>
   <joint name="floor_to_platform" type="fixed">
@@ -92,5 +92,5 @@
   </joint>
   <!-- Camera Calibration-->
-  <xacro:property name="camera_cal" value="${load_yaml('$(find snp_blending)/config/camera_calibration.yaml')}" />
+  <xacro:property name="camera_cal" value="${load_yaml('$(find snp_blending)/config/calibration.yaml')}" />
   <link name="camera_color_optical_frame"/>
   <joint name="tool0_to_camera" type="fixed">

Commit message: Fixed issue in snp_blending URDF (#69)

File: snp_blending/urdf/pushcorp.xacro (robot description, xacro)
@@ -5,5 +5,5 @@
     <xacro:property name="media_radius" value="${2 * 0.0254}"/>
     <xacro:property name="chuck_length" value="0.055"/>
-    <xacro:property name="chuck_radius" value="${1.0 * 0.0254}}"/>
+    <xacro:property name="chuck_radius" value="${1.0 * 0.0254}"/>
     <link name="${prefix}base">
       <visual>
